File: Mote_switch/Mote_switch.brd (EAGLE design)
At the start: 91.1 x 49.5 mm, 21 parts, among them J1 CON_TERMINAL_BLOCK_02-5MM, J2 CON_TERMINAL_BLOCK_03-5MM, J3 CON_TERMINAL_BLOCK_02-5MM, J4 CON_TERMINAL_BLOCK_03-5MM, J5 CON_TERMINAL_BLOCK_02-5MM, J6 CON_TERMINAL_BLOCK_02-5MM, K1 JW1C, K2 JW1C

Commit message: Schematics updated
Parts:
- moved R4 10.9 mm to (48.3, 10.2)
- moved R1 2.54 mm to (74.9, 20.3)
- moved T1 1.27 mm to (40.6, 14.0)
- moved T2 1.27 mm to (40.6, 24.1)
Routing:
- net N$6: track 34.6 -> 17.7 mm
- net D3: track 47.6 -> 37.3 mm, vias 0 -> 1
- net VCC: track 119.3 -> 109.1 mm, vias 1 -> 2
- net N$2: track 17.0 -> 12.3 mm, vias 2 -> 0
- net N$9: track 37.3 -> 33.2 mm
- net N$1: track 22.4 -> 20.3 mm
- net N$7: track 6.30 -> 7.57 mm
- net N$5: track 5.26 -> 6.53 mm
- net GND: track 101.6 -> 102.4 mm
- net N$10: track 26.3 -> 25.7 mm
- net N$11: track 42.6 -> 43.0 mm, vias 1 -> 0
