File: Mote_RgbLedStrip/Mote_RgbLedStripController.sch (EAGLE design)
At the start: 3 parts, among them J1 CON_TERMINAL_BLOCK_02-5MM

Commit message: * Mote_RgbLedStrip - Pin configuration has changed + Mote_irSender + IRrecord * GatewayBase - Added support for AC controller
Parts:
- added Q1, Q2, Q3: 2N2222A, transistor-npn:2N2222A
Connections:
- new net IN_B: Q3.C
- new net IN_G: Q2.C
- new net IN_R: Q1.C
- net D3: now also Q1.B
- net D6: now also Q3.B
- net D9: now also Q2.B
- net GND: now also Q1.E, Q2.E, Q3.E
